File: pcb/wifimeter.kicad_pcb (KiCad board)
At the start: 2 copper layers, 19.6 x 26.2 mm, 28 parts, among them P1 CONN, P2 BATT, U1 BD47xx, U2 ESP8266, U3 MIC550x, U4 Flash, U5 LM358, X1 26MHz

Commit message: pcb: Add version to silkscreen
Other:
- board text added: "v1.0"
